File: PCB_Files/STM_PLC_Board/STM_PLC_Board.kicad_sch (KiCad schematic)
At the start: 0 parts

Commit message: new
Parts:
- added U1: STM32F446RETx, Package_QFP:LQFP-64_10x10mm_P0.5mm, symbol MCU_ST_STM32F4:STM32F446RETx
Connections:
- new net: U1.18 (VSS), U1.31 (VSS), U1.47 (VSS), U1.63 (VSS)
Changed lines of the file:
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@@
 	(generator_version "10.0")
 	(paper "A4")
+	(symbol
+		(lib_id "MCU_ST_STM32F4:STM32F446RETx")
+		(at 78.74 78.74 0)
+		(unit 1)
+		(body_style 1)
+		(exclude_from_sim no)
+		(in_bom yes)
+		(on_board yes)
+		(in_pos_files yes)
+		(dnp no)
+		(fields_autoplaced yes)
+		(property "Reference" "U1"
+			(at 83.4233 124.46 0)
+			(show_name no)
+			(do_not_autoplace no)
+			(effects
+				(font
+					(size 1.27 1.27)
+				)
+				(justify left)
+			)
+		)
+		(property "Value" "STM32F446RETx"
+			(at 83.4233 127 0)
+			(show_name no)
+			(do_not_autoplace no)
+			(effects
+				(font
+					(size 1.27 1.27)
+				)
+				(justify left)
+			)
+		)
+		(property "Footprint" "Package_QFP:LQFP-64_10x10mm_P0.5mm"
+			(at 60.96 121.92 0)
+			(hide yes)
+			(show_name no)
+			(do_not_autoplace no)
+			(effects
+				(font
+					(size 1.27 1.27)
+				)
+				(justify right)
+			)
+		)
+		(property "Datasheet" "https://www.st.com/resource/en/datasheet/stm32f446re.pdf"
+			(at 78.74 78.74 0)
+			(hide yes)
+			(show_name no)
+			(do_not_autoplace no)
+			(effects
+				(font
+					(size 1.27 1.27)
+				)
+			)
+		)
+		(property "Description" "STMicroelectronics Arm Cortex-M4 MCU, 512KB flash, 128KB RAM, 180 MHz, 1.8-3.6V, 50 GPIO, LQFP64"
+			(at 78.74 78.74 0)
+			(hide yes)
+			(show_name no)
+			(do_not_autoplace no)
+			(effects
+				(font
+					(size 1.27 1.27)
+				)
+			)
+		)
+		(pin "31"
+		)
+		(pin "59"
+		)
+		(pin "56"
+		)
+		(pin "4"
+		)
+		(pin "33"
+		)
+		(pin "61"
+		)
+		(pin "62"
+		)
+		(pin "16"
+		)
+		(pin "64"
+		)
+		(pin "55"
+		)
+		(pin "60"
+		)
+		(pin "48"
+		)
+		(pin "32"
+		)
+		(pin "57"
+		)
+		(pin "6"
+		)
+		(pin "9"
+		)
+		(pin "34"
+		)
+		(pin "7"
+		)
+		(pin "10"
+		)
+		(pin "8"
+		)
+		(pin "3"
+		)
+		(pin "5"
+		)
+		(pin "2"
+		)
+		(pin "1"
+		)
+		(pin "17"
+		)
+		(pin "21"
+		)
+		(pin "25"
+		)
+		(pin "44"
+		)
+		(pin "42"
+		)
+		(pin "11"
+		)
+		(pin "22"
+		)
+		(pin "35"
+		)
+		(pin "36"
+		)
+		(pin "37"
+		)
+		(pin "50"
+		)
+		(pin "38"
+		)
+		(pin "43"
+		)
+		(pin "18"
+		)
+		(pin "20"
+		)
+		(pin "30"
+		)
+		(pin "47"
+		)
+		(pin "52"
+		)
+		(pin "46"
+		)
+		(pin "40"
+		)
+		(pin "39"
+		)
+		(pin "15"
+		)
+		(pin "12"
+		)
+		(pin "24"
+		)
+		(pin "45"
+		)
+		(pin "14"
+		)
+		(pin "41"
+		)
+		(pin "23"
+		)
+		(pin "13"
+		)
+		(pin "49"
+		)
+		(pin "19"
+		)
+		(pin "27"
+		)
+		(pin "58"
+		)
+		(pin "51"
+		)
+		(pin "26"
+		)
+		(pin "63"
+		)
+		(pin "53"
+		)
+		(pin "29"
+		)
+		(pin "54"
+		)
+		(pin "28"
+		)
+		(instances
+			(project "STM_PLC_Board"
+				(path "/ba7311af-3053-4b06-bf5c-d2742cc73435"
+					(reference "U1")
+					(unit 1)
+				)
+			)
+		)
+	)
 	(sheet_instances
 		(path "/"
