File: Digital_Board/STM_PLC_Board/stm32_st8500.kicad_sch (KiCad schematic)
At the start: 31 parts

Commit message: schematic done
Parts:
- removed R? (x2): 0R, symbol Device:R_Small
- added C?: 1uF, symbol Device:C
- added J?: Conn_02x06_Odd_Even, symbol Connector_Generic:Conn_02x06_Odd_Even
- added R? (x2): 0R, symbol Device:R_Small
Connections:
- net USART3_RXD is gone; now on net PLC_HOST_USART3_RXD: R?.2
- net USART3_TXD is gone; now on net PLC_HOST_USART3_TXD: R?.1
- net +3.3V: now also J?.2 (Pin_2)
- net DBG_USART2_RTS: now also R?.2
- net DBG_USART2_RX: now also U?.50 (GPIO01_4), R?.2
- net DBG_USART2_TX: now also U?.49 (GPIO01_5)
- net GND: now also C?.2, J?.1 (Pin_1)
- net at J?.14 (Pin_14): now also R?.1
- net at C?.2, R?.2, U?.23 (AVDD_3V3_AFE): now also U?.28 (DVDD_3V3_IO), C?.1
- net PLC_JTDI: now reaches J?.12 (Pin_12)
- net PLC_JTDI: now also U?.38 (GPIO03_7)
- net PLC_JTDO: now reaches J?.10 (Pin_10)
- net PLC_JTDO: now also U?.40 (GPIO03_5)
- net at J?.16 (Pin_16): now also R?.1
- net PLC_JTCK: now reaches J?.7 (Pin_7)
- net PLC_JTCK: now also U?.41 (GPIO03_4)
- net PLC_JTMS: now reaches J?.8 (Pin_8)
- net PLC_JTMS: now also U?.42 (GPIO03_3)
- net PLC_JRST: now reaches J?.9 (Pin_9)
- net PLC_JRST: now also U?.39 (GPIO03_6)
- net GPIO00_7: now reaches U?.29 (GPIO00_7)
- net GPIO00_6: now reaches U?.30 (GPIO00_6)
- net PLC_HOST_USART3_TXD: now reaches U?.31 (GPIO00_5)
- net PLC_HOST_USART3_RXD: now reaches U?.32 (GPIO00_4)
- net SPI3_MISO: now reaches U?.33 (GPIO00_3)
- net SPI3_MISO: now also J?.9 (Pin_9)
- net SPI3_NSS: now reaches U?.34 (GPIO00_2)
- net SPI3_NSS: now also J?.5 (Pin_5)
- net SPI3_MOSI: now reaches U?.35 (GPIO00_1)
- net SPI3_MOSI: now also J?.11 (Pin_11)
- net SPI3_SCK: now reaches U?.36 (GPIO00_0)
- net SPI3_SCK: now also J?.7 (Pin_7)
- net BAND_SEL: now reaches U?.47 (GPIO01_7)
- net GPIO01_6: now reaches U?.48 (GPIO01_6)
- net USART3_CTS renamed PLC_HOST_USART3_CTS
- net USART3_RTS renamed PLC_HOST_USART3_RTS
- new net I2C1_SCL: J?.10 (Pin_10)
- new net I2C1_SDA: J?.12 (Pin_12)
- no-connect marks 18 -> 22
Other:
- note added: "Do we need SFlash?"
- note added: "Micellaneous (Analog)"
- note added: "ZeroC"
- moved on the sheet: R?
