File: Digital_Board/STM_PLC_Board/components.kicad_sch (KiCad schematic)
At the start: 42 parts, among them J2 Conn_02x14_Odd_Even, Q1 2N7002, Q2 2N7002, Q3 2N7002, Q4 2N7002, SW1 SW_Push, SW2 SW_DIP_x01, SW3 SW_DIP_x01

Commit message: schematic done
Parts:
- removed J2: Conn_02x14_Odd_Even, symbol Connector_Generic:Conn_02x14_Odd_Even
- removed R11, R12, R13, R14, R15, R16, R17, R18, R19, R20, R21: 0R, symbol Device:R_Small
- removed R22: 10k, symbol Device:R_Small
- removed TP1, TP2, TP3, TP4: TestPoint, symbol Connector:TestPoint
- added J?: Conn_02x14_Odd_Even_Female, symbol Connector_Generic:Conn_02x14_Odd_Even
- added J?: JTAG Connector, symbol Connector_Generic:Conn_02x10_Odd_Even
- added R? (x3): 10k, symbol Device:R
- added R? (x11): 0R, symbol Device:R_Small
- added R?: 0R, symbol Device:R
- added R?: 10k, symbol Device:R_Small
- added TP? (x2): TestPoint, symbol Connector:TestPoint
Connections:
- net +3.3V: now also J?.1 (Pin_1), R?.1
- net DBG_USART2_CTS: now also R?.1
- net DBG_USART2_RTS: now also R?.2
- net DBG_USART2_RX: now also R?.2
- net DBG_USART2_TX: now also R?.1
- net GND: now also J?.10 (Pin_10), J?.12 (Pin_12), J?.14 (Pin_14), J?.16 (Pin_16), J?.18 (Pin_18), J?.2 (Pin_2), J?.20 (Pin_20), J?.26 (Pin_26), J?.28 (Pin_28), J?.4 (Pin_4), J?.6 (Pin_6), J?.8 (Pin_8), R?.1
- net PLC_BOOT0: now also J?.4 (Pin_4), TP?.1
- net PLC_BOOT1: now also R?.2
- net PLC_BOOT2: now also J?.3 (Pin_3), TP?.1
- net PLC_LPMODE: now also R?.1
- net PLC_RST: now also R?.1, R?.1, R?.2
- net VDC_LD: now also J?.25 (Pin_25), J?.27 (Pin_27)
- new net: J?.21 (Pin_21), R?.2
- new net: J?.11 (Pin_11), R?.2
- new net: J?.13 (Pin_13), R?.2
- new net: J?.14 (Pin_14), R?.1
- new net: J?.16 (Pin_16), R?.1
- new net: J?.17 (Pin_17), R?.2
- new net: J?.18 (Pin_18), R?.1
- new net: J?.19 (Pin_19), R?.2
- new net: J?.20 (Pin_20), R?.1
- new net: J?.23 (Pin_23), R?.2
- new net: J?.6 (Pin_6), R?.1
- new net: J?.15 (Pin_15), R?.2
- new net +3V3: J?.1 (Pin_1), J?.2 (Pin_2), R?.1, R?.1
- new net PLC_HOST_USART3_CTS: R?.1
- new net PLC_HOST_USART3_RTS: R?.2
- new net PLC_HOST_USART3_RXD: R?.2
- new net PLC_HOST_USART3_TXD: R?.1
- new net PLC_JRST: J?.3 (Pin_3), J?.9 (Pin_9), R?.2
- new net PLC_JTCK: J?.7 (Pin_7), J?.9 (Pin_9), R?.2
- new net PLC_JTDI: J?.12 (Pin_12), J?.5 (Pin_5)
- new net PLC_JTDO: J?.10 (Pin_10), J?.13 (Pin_13), R?.2
- new net PLC_JTMS: J?.7 (Pin_7), J?.8 (Pin_8)
Other:
- note added: "JTAG Connector"
- note added: "ST8500 to STM32 (Analog)"
- note removed: "STM32 to ST8500 (Digital)"

Commit message: added components
Parts:
- C15, C16: renamed from C?; footprint (none) -> DigitalBoardLibrary:0805 Capacitor SMD
- C9: footprint (none) -> DigitalBoardLibrary:0805 Capacitor SMD
- R11, R12, R13, R14, R15, R16, R17, R18, R19, R20, R21, R22, R23, R24, R25, R26, R27: renamed from R?; footprint (none) -> DigitalBoardLibrary:0805 SMD Resistor
- R2, R3, R4, R5, R6, R7, R8: footprint (none) -> DigitalBoardLibrary:0805 SMD Resistor
- gave numbers to parts that had none: 7

Commit message: components?
Parts:
- J4: footprint (none) -> DigitalBoardLibrary:JTAG_CONN10_SHF_12P7X5P08_SAI
Changed lines of the file:
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@@
 			)
 		)
-		(property "Footprint" ""
+		(property "Footprint" "DigitalBoardLibrary:JTAG_CONN10_SHF_12P7X5P08_SAI"
 			(at 123.19 162.56 0)
 			(hide yes)

Commit message: pcb changes
Parts:
- removed J4: JTAG Connector, DigitalBoardLibrary:JTAG_CONN10_SHF_12P7X5P08_SAI, symbol Connector_Generic:Conn_02x10_Odd_Even
- added D6: SM6T18A, DigitalBoardLibrary:SMB_STM-M, symbol Diode:SM6T18A
- added J4: JTAG_10CON, DigitalBoardLibrary:CONN10_SHF_12P7X5P08_SAI, symbol Digital_Mesh:JTAG_10CON
- added J5: 3pin_61300311121, DigitalBoardLibrary:3PIN_HEADER, symbol Digital_Mesh:3pin_61300311121
- added J6: ViperJACK, DigitalBoardLibrary:ViperJACK_0022152046, symbol Connector:Conn_01x04_Pin
- added J7: Barrel_Jack_Switch, DigitalBoardLibrary:jack_694106301002, symbol Connector:Barrel_Jack_Switch
- added R28: 0R, DigitalBoardLibrary:0805 SMD Resistor, symbol Device:R_Small
- D1, D2, D3, D4, D5: footprint (none) -> DigitalBoardLibrary:GREENLED_598-8170_DIA
- J2: value Conn_02x06_Odd_Even -> Misc_STM32_Conn; footprint (none) -> DigitalBoardLibrary:2x6_FemaleHeader
- J3: footprint (none) -> DigitalBoardLibrary:2x14_FemaleHeaderSAMESKY_SSK04-FPH-254-B14
- Q1, Q2, Q3, Q4: footprint Package_TO_SOT_SMD:SOT-23 -> DigitalBoardLibrary:MOSFET_SOT-23TO-236_318-08_ONS
- SW1, SW2, SW3: footprint (none) -> DigitalBoardLibrary:SWITCH_CL-SB-12A-01T_NDC
- U2: footprint Package_TO_SOT_SMD:SOT-223-3_TabPin2 -> DigitalBoardLibrary:VoltageRegulator_SOT_AMS_ADS
Connections:
- net PLC_BOOT2 is gone; now on net GND: J3.3 (Pin_3), TP1.1
- net +3.3V: now also J6.1 (Pin_1)
- net +3V3: now also J4.1
- net GND: now also D6.1 (A1), J6.2 (Pin_2), J7.2
- net PLC_JRST: now also J4.2
- net PLC_JTCK: now also J4.5
- net PLC_JTDI: now also J4.3
- net PLC_JTDO: now also J4.7
- net PLC_JTMS: now also J4.4
- net VBUS: now also D6.2 (A2), J5.2, R28.1
- net VDC_LD: now also R28.2
- net at R25.2: now also J4.8
- new net: J5.1, J6.3 (Pin_3)
- new net: J5.3, J7.1
- no-connect marks 11 -> 13
Other:
- note added: "DC Supply Voltage"
- note added: "JACK POWER Black BOX : +12V"
- note added: "POWER from PSU ( VIPER BOARD ) VDC_CON : +12V/+15V 3V3_CON : +3.3V"
- note added: "STM32 to ST8500"
- note removed: "ST8500 to STM32 (Analog)"
